File: PCBs/hp141t-emulator-system/v02/emulator-pcb/emulator-pcb.kicad_sch (KiCad schematic)
At the start: 49 parts, among them J1 Conn_Coaxial, J2 Conn_Coaxial, J3 Conn_Coaxial, J4 Mini-DIN-5, Q1 2N2222, U1 LM358, U2 XR2206CP, U3 XR2206CP

Commit message: Removed voltage divider. Added 0.1uF power capacitors.
Parts:
- removed R28: 33k, Resistor_THT:R_Axial_DIN0207_L6.3mm_D2.5mm_P7.62mm_Horizontal, symbol Device:R
- removed R29: 10k, Resistor_THT:R_Axial_DIN0207_L6.3mm_D2.5mm_P7.62mm_Horizontal, symbol Device:R
- added C10, C9: 0.1uF, Capacitor_THT:C_Axial_L3.8mm_D2.6mm_P7.50mm_Horizontal, symbol Device:C
- R27: value 100k -> 2.2k
Connections:
- net -12V: now also C10.2
- net GND: now also C10.1, C9.2
- net at S1.2: now also J4.4, C9.1
